File: PCB/RSSQ.kicad_sch (KiCad schematic)
At the start: 0 parts

Commit message: Added various parts to schematic
Other:
- added sheet ESP8285 (ESP8285.kicad_sch)
- added sheet Keyboard (Keyboard.kicad_sch)
- added sheet USB-C (USB-C.kicad_sch)
- added sheet nRF52840 (nRF52840.kicad_sch)
Changed lines of the file:
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@@
 	(generator_version "9.0")
 	(paper "A4")
+	(sheet
+		(at 145.415 55.245)
+		(size 55.88 25.4)
+		(exclude_from_sim no)
+		(in_bom yes)
+		(on_board yes)
+		(dnp no)
+		(fields_autoplaced yes)
+		(stroke
+			(width 0.1524)
+			(type solid)
+		)
+		(fill
+			(color 0 0 0 0.0000)
+		)
+		(property "Sheetname" "ESP8285"
+			(at 145.415 54.5334 0)
+			(effects
+				(font
+					(size 1.27 1.27)
+				)
+				(justify left bottom)
+			)
+		)
+		(property "Sheetfile" "ESP8285.kicad_sch"
+			(at 145.415 81.2296 0)
+			(effects
+				(font
+					(size 1.27 1.27)
+				)
+				(justify left top)
+			)
+		)
+		(instances
+			(project "RSSQ"
+				(path "/e9cd8552-a55f-4a0c-81be-0de8f48f955a"
+					(page "3")
+				)
+			)
+		)
+	)
+	(sheet
+		(at 59.69 47.625)
+		(size 37.465 15.24)
+		(exclude_from_sim no)
+		(in_bom yes)
+		(on_board yes)
+		(dnp no)
+		(fields_autoplaced yes)
+		(stroke
+			(width 0.1524)
+			(type solid)
+		)
+		(fill
+			(color 0 0 0 0.0000)
+		)
+		(property "Sheetname" "USB-C"
+			(at 59.69 46.9134 0)
+			(effects
+				(font
+					(size 1.27 1.27)
+				)
+				(justify left bottom)
+			)
+		)
+		(property "Sheetfile" "USB-C.kicad_sch"
+			(at 59.69 63.4496 0)
+			(effects
+				(font
+					(size 1.27 1.27)
+				)
+				(justify left top)
+			)
+		)
+		(instances
+			(project "RSSQ"
+				(path "/e9cd8552-a55f-4a0c-81be-0de8f48f955a"
+					(page "5")
+				)
+			)
+		)
+	)
+	(sheet
+		(at 145.415 90.805)
+		(size 64.77 26.67)
+		(exclude_from_sim no)
+		(in_bom yes)
+		(on_board yes)
+		(dnp no)
+		(fields_autoplaced yes)
+		(stroke
+			(width 0.1524)
+			(type solid)
+		)
+		(fill
+			(color 0 0 0 0.0000)
+		)
+		(property "Sheetname" "Keyboard"
+			(at 145.415 90.0934 0)
+			(effects
+				(font
+					(size 1.27 1.27)
+				)
+				(justify left bottom)
+			)
+		)
+		(property "Sheetfile" "Keyboard.kicad_sch"
+			(at 145.415 118.0596 0)
+			(effects
+				(font
+					(size 1.27 1.27)
+				)
+				(justify left top)
+			)
+		)
+		(instances
+			(project "RSSQ"
+				(path "/e9cd8552-a55f-4a0c-81be-0de8f48f955a"
+					(page "4")
+				)
+			)
+		)
+	)
+	(sheet
+		(at 144.78 29.21)
+		(size 53.34 16.51)
+		(exclude_from_sim no)
+		(in_bom yes)
+		(on_board yes)
+		(dnp no)
+		(fields_autoplaced yes)
+		(stroke
+			(width 0.1524)
+			(type solid)
+		)
+		(fill
+			(color 0 0 0 0.0000)
+		)
+		(property "Sheetname" "nRF52840"
+			(at 144.78 28.4984 0)
+			(effects
+				(font
+					(size 1.27 1.27)
+				)
+				(justify left bottom)
+			)
+		)
+		(property "Sheetfile" "nRF52840.kicad_sch"
+			(at 144.78 46.3046 0)
+			(effects
+				(font
+					(size 1.27 1.27)
+				)
+				(justify left top)
+			)
+		)
+		(instances
+			(project "RSSQ"
+				(path "/e9cd8552-a55f-4a0c-81be-0de8f48f955a"
+					(page "2")
+				)
+			)
+		)
+	)
 	(sheet_instances
 		(path "/"
